File: Testinium_puro_humidor/Testinium_puro_humidor/Testinium_puro_humidor.kicad_sch (KiCad schematic)
At the start: 4 parts

Commit message: fan , uv led ,regülator devresi eklendi. piezo ve sarj devresi kaldi
Changed lines of the file:
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@@
 	)
 	(sheet
-		(at 95.25 30.48)
+		(at 63.5 38.1)
 		(size 30.48 15.24)
 		(exclude_from_sim no)
@@
 		)
 		(property "Sheetname" "sarj"
-			(at 95.25 29.7684 0)
+			(at 63.5 37.3884 0)
 			(effects
 				(font
@@
 		)
 		(property "Sheetfile" "sarj.kicad_sch"
-			(at 95.25 46.3046 0)
+			(at 63.5 53.9246 0)
 			(effects
 				(font
@@
 	)
 	(sheet
-		(at 54.61 26.67)
-		(size 29.21 22.86)
+		(at 104.14 38.1)
+		(size 29.21 15.24)
 		(exclude_from_sim no)
 		(in_bom yes)
@@
 		)
 		(property "Sheetname" "regulator"
-			(at 54.61 25.9584 0)
+			(at 104.14 37.3884 0)
 			(effects
 				(font
@@
 		)
 		(property "Sheetfile" "regulator.kicad_sch"
-			(at 54.61 50.1146 0)
+			(at 104.14 53.9246 0)
 			(effects
 				(font
@@
 		)
 		(pin "3V3" input
-			(at 83.82 38.1 0)
+			(at 133.35 41.91 0)
 			(effects
 				(font

Commit message: sematik tamamlandi
Parts:
- added BZ1: Buzzer, symbol Device:Buzzer
- added H1, H2, H3: MountingHole_Pad_MP, MountingHole:MountingHole_3.2mm_M3_Pad, symbol Mechanical:MountingHole_Pad_MP
- added JP1: piezzo_jump, symbol Jumper:Jumper_3_Bridged12
- added JP2: uv_jump, symbol Jumper:Jumper_3_Bridged12
- D1, D2: footprint (none) -> LED_SMD:LED_0805_2012Metric
- R1, R2: footprint (none) -> Resistor_SMD:R_0805_2012Metric
Connections:
- new net 5V: JP1.3 (B), JP2.3 (B)
- new net Power: JP1.1 (A), JP2.1 (A)
- new net piezzo_vcc: JP1.2 (C)
- new net uvled/UV_VCC: JP2.2 (C)
Other:
- removed sheet sarj
- sheet ESP32 ports: added ESP32_3V3, I2C0_SCL, I2C0_SDA, I2C1_SCL, I2C1_SDA; removed none
- sheet FAN1 ports: added Fan_VCC; removed FAN1_Enable
- sheet FAN2 ports: added Fan_VCC; removed FAN2_Enable
- sheet oled ports: added none; removed Oled_3V3, Oled_GND
- sheet piezzo ports: added MCU_Piezzo, Piezzo_Vcc; removed none
- sheet regulator ports: added 3V3_esp32, 5V, 7V4; removed 3V3
- sheet sht31 ports: added none; removed Sht31_3V3, Sht31_GND
- sheet uvled ports: added MCU_UV, UV_VCC; removed none
- moved on the sheet: D1, D2, R1, R2
