File: Testinium_puro_humidor/Testinium_puro_humidor/piezzo.kicad_sch (KiCad schematic)
At the start: 0 parts

Commit message: fan , uv led ,regülator devresi eklendi. piezo ve sarj devresi kaldi
Parts:
- added J3: Piezzo, Connector_JST:JST_EH_B2B-EH-A_1x02_P2.50mm_Vertical, symbol Connector:Conn_01x02_Pin
Connections:
- new net GND: J3.2 (Pin_2)
Changed lines of the file:
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@@
 	(generator_version "9.0")
 	(paper "A4")
+	(wire
+		(pts
+			(xy 43.18 62.23) (xy 43.18 49.53)
+		)
+		(stroke
+			(width 0)
+			(type default)
+		)
+	)
+	(symbol
+		(lib_id "Connector:Conn_01x02_Pin")
+		(at 38.1 46.99 0)
+		(unit 1)
+		(exclude_from_sim no)
+		(in_bom yes)
+		(on_board yes)
+		(dnp no)
+		(fields_autoplaced yes)
+		(property "Reference" "J3"
+			(at 38.735 41.91 0)
+			(effects
+				(font
+					(size 1.27 1.27)
+				)
+			)
+		)
+		(property "Value" "Piezzo"
+			(at 38.735 44.45 0)
+			(effects
+				(font
+					(size 1.27 1.27)
+				)
+			)
+		)
+		(property "Footprint" "Connector_JST:JST_EH_B2B-EH-A_1x02_P2.50mm_Vertical"
+			(at 38.1 46.99 0)
+			(effects
+				(font
+					(size 1.27 1.27)
+				)
+				(hide yes)
+			)
+		)
+		(property "Datasheet" "~"
+			(at 38.1 46.99 0)
+			(effects
+				(font
+					(size 1.27 1.27)
+				)
+				(hide yes)
+			)
+		)
+		(property "Description" "Generic connector, single row, 01x02, script generated"
+			(at 38.1 46.99 0)
+			(effects
+				(font
+					(size 1.27 1.27)
+				)
+				(hide yes)
+			)
+		)
+		(pin "1"
+		)
+		(pin "2"
+		)
+		(instances
+			(project "Testinium_puro_humidor"
+				(path "/eaf24445-473d-4e1b-a90d-ef2c4a02e74f/745420fc-bc35-43f3-afbe-dcd060b32210"
+					(reference "J3")
+					(unit 1)
+				)
+			)
+		)
+	)
+	(symbol
+		(lib_id "power:GND")
+		(at 43.18 62.23 0)
+		(unit 1)
+		(exclude_from_sim no)
+		(in_bom yes)
+		(on_board yes)
+		(dnp no)
+		(fields_autoplaced yes)
+		(property "Reference" "#PWR07"
+			(at 43.18 68.58 0)
+			(effects
+				(font
+					(size 1.27 1.27)
+				)
+				(hide yes)
+			)
+		)
+		(property "Value" "GND"
+			(at 43.18 67.31 0)
+			(effects
+				(font
+					(size 1.27 1.27)
+				)
+			)
+		)
+		(property "Footprint" ""
+			(at 43.18 62.23 0)
+			(effects
+				(font
+					(size 1.27 1.27)
+				)
+				(hide yes)
+			)
+		)
+		(property "Datasheet" ""
+			(at 43.18 62.23 0)
+			(effects
+				(font
+					(size 1.27 1.27)
+				)
+				(hide yes)
+			)
+		)
+		(property "Description" "Power symbol creates a global label with name \"GND\" , ground"
+			(at 43.18 62.23 0)
+			(effects
+				(font
+					(size 1.27 1.27)
+				)
+				(hide yes)
+			)
+		)
+		(pin "1"
+		)
+		(instances
+			(project "Testinium_puro_humidor"
+				(path "/eaf24445-473d-4e1b-a90d-ef2c4a02e74f/745420fc-bc35-43f3-afbe-dcd060b32210"
+					(reference "#PWR07")
+					(unit 1)
+				)
+			)
+		)
+	)
 )

Commit message: sematik tamamlandi
Parts:
- added C15, C16: 47nF, Capacitor_SMD:C_0805_2012Metric, symbol Device:C
- added D8: GreenLed, LED_SMD:LED_0805_2012Metric, symbol Device:LED
- added D9: D, Diode_SMD:D_SMA, symbol Device:D
- added L1: 100mH, Inductor_SMD:L_10.4x10.4_H4.8, symbol Device:L
- added Q2: 2SC5200, Package_TO_SOT_THT:TO-92_Inline, symbol Transistor_BJT:2SC1815
- added R21: 2K2, Resistor_SMD:R_0805_2012Metric, symbol Device:R
- added R22: 4R7, Resistor_SMD:R_0805_2012Metric, symbol Device:R
- added R23: 330R, Resistor_SMD:R_0603_1608Metric, symbol Device:R
- added R24: 100R, Resistor_SMD:R_0603_1608Metric, symbol Device:R
- added U5: PC817, Package_SO:SOP-4_3.8x4.1mm_P2.54mm, symbol Isolator:PC817
Connections:
- net GND: now also D9.1 (K), L1.2, Q2.2 (C), R24.1
- net piezzo_pin1: now reaches J3.1 (Pin_1)
- net piezzo_pin1: now also C15.1
- new net: C16.1, L1.1, Q2.1 (E)
- new net: Q2.3 (B), R22.2
- new net: C15.2, C16.2, R21.2, R22.1
- new net: D8.2 (A), U5.2
- new net: R23.2, U5.1
- new net: R24.2, U5.3
- new net 3V3: R23.1
- new net MCU_Piezzo: D8.1 (K)
- new net Piezzo_+: D9.2 (A), R21.1, U5.4
Other:
- moved on the sheet: J3
