File: Testinium_puro_humidor/Testinium_puro_humidor/uvled.kicad_sch (KiCad schematic)
At the start: 0 parts

Commit message: fan , uv led ,regülator devresi eklendi. piezo ve sarj devresi kaldi
Parts:
- added D5: GreenLed, LED_SMD:LED_0805_2012Metric, symbol Device:LED
- added D6: D, symbol Device:D
- added J5: Conn_01x02_Fan1, Connector_JST:JST_EH_B2B-EH-A_1x02_P2.50mm_Vertical, symbol Connector:Conn_01x02_Pin
- added Q1: 2N3904, Package_TO_SOT_SMD:SOT-23, symbol Transistor_BJT:2N3904
- added R5, R6: 100R, Resistor_SMD:R_0603_1608Metric, symbol Device:R
- added U4: PC817, Package_SO:SOP-4_3.8x4.1mm_P2.54mm, symbol Isolator:PC817
Connections:
- new net: R5.2, U4.1
- new net: D5.2 (A), U4.2
- new net: R6.2, U4.3
- new net: Q1.2 (B), R6.1
- new net 3V3: J5.1 (Pin_1), R5.1
- new net GND: J5.2 (Pin_2), Q1.1 (E)
- new net MCU_UV: D5.1 (K)
- new net UV_LED_+: D6.1 (K), D6.2 (A), Q1.3 (C), U4.4

Commit message: sematik tamamlandi
Parts:
- D6: footprint (none) -> Diode_SMD:D_SMA
- J5: value Conn_01x02_Fan1 -> Conn_01x02_UV_LED
Connections:
- net 3V3: no longer J5.1 (Pin_1)
- net GND: no longer J5.2 (Pin_2)
- net UV_LED_+: now also J5.1 (Pin_1), J5.2 (Pin_2)
Other:
- moved on the sheet: J5
Changed lines of the file:
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@@
 	(wire
 		(pts
-			(xy 30.48 20.32) (xy 26.67 20.32)
+			(xy 30.48 17.78) (xy 24.13 17.78)
 		)
 		(stroke
@@
 	(wire
 		(pts
-			(xy 30.48 22.86) (xy 26.67 22.86)
+			(xy 30.48 20.32) (xy 24.13 20.32)
 		)
 		(stroke
@@
 			(width 0)
 			(type default)
+		)
+	)
+	(global_label "UV_LED_+"
+		(shape input)
+		(at 30.48 20.32 0)
+		(fields_autoplaced yes)
+		(effects
+			(font
+				(size 1.27 1.27)
+			)
+			(justify left)
+		)
+		(property "Intersheetrefs" "${INTERSHEET_REFS}"
+			(at 42.839 20.32 0)
+			(effects
+				(font
+					(size 1.27 1.27)
+				)
+				(justify left)
+				(hide yes)
+			)
 		)
 	)
@@
 		(property "Intersheetrefs" "${INTERSHEET_REFS}"
 			(at 91.099 25.4 0)
+			(effects
+				(font
+					(size 1.27 1.27)
+				)
+				(justify left)
+				(hide yes)
+			)
+		)
+	)
+	(global_label "3V3"
+		(shape input)
+		(at 31.75 27.94 180)
+		(fields_autoplaced yes)
+		(effects
+			(font
+				(size 1.27 1.27)
+			)
+			(justify right)
+		)
+		(property "Intersheetrefs" "${INTERSHEET_REFS}"
+			(at 25.2572 27.94 0)
+			(effects
+				(font
+					(size 1.27 1.27)
+				)
+				(justify right)
+				(hide yes)
+			)
+		)
+	)
+	(global_label "UV_LED_+"
+		(shape input)
+		(at 30.48 17.78 0)
+		(fields_autoplaced yes)
+		(effects
+			(font
+				(size 1.27 1.27)
+			)
+			(justify left)
+		)
+		(property "Intersheetrefs" "${INTERSHEET_REFS}"
+			(at 42.839 17.78 0)
 			(effects
 				(font
@@
 		(shape input)
 		(at 74.93 24.13 90)
-		(effects
-			(font
-				(size 1.27 1.27)
-			)
-			(justify left)
-		)
-	)
-	(hierarchical_label "3V3"
-		(shape input)
-		(at 31.75 27.94 180)
-		(effects
-			(font
-				(size 1.27 1.27)
-			)
-			(justify right)
-		)
-	)
-	(hierarchical_label "3V3"
-		(shape input)
-		(at 30.48 20.32 0)
 		(effects
 			(font
@@
 	(symbol
 		(lib_id "Connector:Conn_01x02_Pin")
-		(at 21.59 20.32 0)
+		(at 19.05 17.78 0)
 		(unit 1)
 		(exclude_from_sim no)
@@
 		(fields_autoplaced yes)
 		(property "Reference" "J5"
-			(at 22.225 15.24 0)
-			(effects
-				(font
-					(size 1.27 1.27)
-				)
-			)
-		)
-		(property "Value" "Conn_01x02_Fan1"
-			(at 22.225 17.78 0)
+			(at 19.685 12.7 0)
+			(effects
+				(font
+					(size 1.27 1.27)
+				)
+			)
+		)
+		(property "Value" "Conn_01x02_UV_LED"
+			(at 19.685 15.24 0)
 			(effects
 				(font
@@
 		)
 		(property "Footprint" "Connector_JST:JST_EH_B2B-EH-A_1x02_P2.50mm_Vertical"
-			(at 21.59 20.32 0)
+			(at 19.05 17.78 0)
 			(effects
 				(font
@@
 		)
 		(property "Datasheet" "~"
-			(at 21.59 20.32 0)
+			(at 19.05 17.78 0)
 			(effects
 				(font
@@
 		)
 		(property "Description" "Generic connector, single row, 01x02, script generated"
-			(at 21.59 20.32 0)
+			(at 19.05 17.78 0)
 			(effects
 				(font
@@
 			)
 		)
-		(property "Footprint" ""
+		(property "Footprint" "Diode_SMD:D_SMA"
 			(at 74.93 31.75 0)
 			(effects
@@
 					(unit 1)
 				)
-			)
-		)
-	)
-	(symbol
-		(lib_id "power:GND")
-		(at 30.48 22.86 90)
-		(unit 1)
-		(exclude_from_sim no)
-		(in_bom yes)
-		(on_board yes)
-		(dnp no)
-		(fields_autoplaced yes)
-		(property "Reference" "#PWR020"
-			(at 36.83 22.86 0)
-			(effects
-				(font
-					(size 1.27 1.27)
-				)
-				(hide yes)
-			)
-		)
-		(property "Value" "GND"
-			(at 34.29 22.8599 90)
-			(effects
-				(font
-					(size 1.27 1.27)
-				)
-				(justify right)
-			)
-		)
-		(property "Footprint" ""
-			(at 30.48 22.86 0)
-			(effects
-				(font
-					(size 1.27 1.27)
-				)
-				(hide yes)
-			)
-		)
-		(property "Datasheet" ""
-			(at 30.48 22.86 0)
-			(effects
-				(font
-					(size 1.27 1.27)
-				)
-				(hide yes)
-			)
-		)
-		(property "Description" "Power symbol creates a global label with name \"GND\" , ground"
-			(at 30.48 22.86 0)
-			(effects
-				(font
-					(size 1.27 1.27)
-				)
-				(hide yes)
-			)
-		)
-		(pin "1"
-		)
-		(instances
-			(project "Testinium_puro_humidor"
-				(path "/eaf24445-473d-4e1b-a90d-ef2c4a02e74f/94b7e529-b722-4dba-bd12-0193f3655d72"
-					(reference "#PWR020")
-					(unit 1)
-				)
